Commit message: Fix for IMU

File: hros5_common/hros5_description/urdf/modules/torso.xacro (robot description, xacro)
@@ -5,5 +5,4 @@
 		<parent link="base_link"/>
 		<child link="torso"/>
-		<origin xyz="0 0 0.24" rpy="0 0 0"/>
 	</joint>
 	<!-- TORSO -->
@@ -17,8 +16,7 @@
 	</link>
 <!-- IMU properties -->
-<!--
-<joint name="imu_joint" type="floating">
-    <parent link="base_link"/>
-    <child link="torso"/>
+<joint name="imu_joint" type="fixed">
+    <parent link="torso"/>
+    <child link="imu_link"/>
     <origin xyz="0.0 0.0 0.033" rpy="0.0 0.0 0.0"/>
 </joint>
@@ -35,5 +33,5 @@
 	<gazebo>
         <plugin filename="libhector_gazebo_ros_imu.so" name="gazebo_ros_imu">
-          <bodyName>torso</bodyName>
+          <bodyName>imu_link</bodyName>
           <updateRate>50</updateRate>
           <serviceName>/hros5/imu_service</serviceName>
@@ -44,4 +42,3 @@
         </plugin>
       </gazebo>
--->
 </robot>
